File: hardware/PUTM_EV_DASHBOARD_SOCKET_2025/PUTM_EV_DASHBOARD_SOCKET_2025.kicad_pcb (KiCad board)
At the start: 2 copper layers, 200 x 150 mm, 59 parts, among them J1pin200000 Conn_02x20_Top_Bottom_Mountin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, J2SO2 Conn_02x20_Top_Bottom_Mountin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, J2SWD2 Conn_01x06_MountingPin, J3CAN0 Conn_01x04_MountingPin, J3CAN2 Conn_01x04_MountingPin, J4POWER0 Conn_01x06_MountingPin, J5POWER1 Conn_01x06_MountingPin, Q4 BSS138, Q5 BSS138, Q6 BSS138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

Commit message: prawie gotowe
Parts:
- removed J2SWD2: Conn_01x06_MountingPin, Connector_PinHeader_1.27mm:PinHeader_1x06_P1.27mm_Vertical
- removed J3CAN0: Conn_01x04_MountingPin, Connector_Molex:Molex_CLIK-Mate_502382-0470_1x04-1MP_P1.25mm_Vertical
- removed J3CAN2: Conn_01x04_MountingPin, Connector_PinHeader_1.27mm:PinHeader_1x04_P1.27mm_Vertical
- removed the J4POWER0 at (83.8, 76.7)
- removed the J5POWER1 at (141.7, 161.3)
- removed the J5POWER1 at (231.9, 82.4)
- removed R6: 1K, Resistor_SMD:R_1206_3216Metric
- removed SW6: SW_Push, Button_Switch_SMD:SW_Push_1TS009xxxx-xxxx-xxxx_6x6x5mm
- added J5POWER1: Conn_01x06_MountingPin, Connector_Wire:SolderWire-0.1sqmm_1x06_P3.6mm_D0.4mm_OD1mm_Relief, F.Cu at (227.6, 111.0)
- ALT_CAN0, AMS1, CS_BTN1, DRS_BTN1, FUSE_LED1, J2SO2, J4POWER0, RTD_BTN1, SAFETY_LED1, SW1, SW2, SW3, SW4, SW5, TERM_0, TERM_1, TSA_BTN1, USR_BTN1: moved to B.Cu
- AMS0: renamed from D10; moved to B.Cu
- CAN0: value Conn_01x04_MountingPin -> Conn_01x09; footprint Connector_Molex:Molex_CLIK-Mate_502382-0470_1x04-1MP_P1.25mm_Vertical -> Connector_Dsub:DSUB-9_Pins_Horizontal_P2.77x2.84mm_EdgePinOffset4.94mm_Housed_MountingHolesOffset4.94mm; moved to B.Cu
- CAN1: footprint Connector_PinHeader_1.27mm:PinHeader_1x04_P1.27mm_Vertical -> Connector_Wire:SolderWire-0.1sqmm_1x04_P3.6mm_D0.4mm_OD1mm_Relief
- FUSE_LED0: renamed from D12; moved to B.Cu
- SAFETY_LED0: renamed from D11; moved to B.Cu
- SWD0: footprint Connector_Dsub:DSUB-9_Pins_Horizontal_P2.77x2.54mm_EdgePinOffset9.40mm -> Connector_Molex:Molex_CLIK-Mate_502382-0670_1x06-1MP_P1.25mm_Vertical; moved to B.Cu
- SWD2: footprint Connector_PinHeader_1.27mm:PinHeader_1x06_P1.27mm_Vertical -> Connector_Wire:SolderWire-0.1sqmm_1x06_P3.6mm_D0.4mm_OD1mm_Relief
- moved USR_BTN1 159.4 mm to (210.8, 28.4)
- moved J4POWER0 156.6 mm to (237.1, 31.4), turned to 180 degrees
- moved SAFETY_LED1 152.3 mm to (204.4, 28.4)
- moved DRS_BTN1 152.0 mm to (207.6, 28.4)
- moved FUSE_LED1 146.7 mm to (201.2, 28.4)
- moved AMS1 146.5 mm to (221.3, 40.5), turned to 180 degrees
- moved TSA_BTN1 145.1 mm to (199.0, 40.5), turned to 180 degrees
- moved RTD_BTN1 142.8 mm to (202.2, 40.5), turned to 180 degrees
- moved J2SO2 136.0 mm to (223.7, 37.1), turned to 90 degrees
- moved CS_BTN1 134.5 mm to (205.4, 40.6), turned to 180 degrees
- moved AMS0 126.0 mm to (109.3, 27.7)
- moved R9 125.7 mm to (109.4, 27.7), turned to 180 degrees
- moved SWD1 124.5 mm to (180.8, 42.7), turned to -90 degrees
- moved SAFETY_LED0 124.4 mm to (109.4, 33.8)
- moved FUSE_LED0 122.8 mm to (109.4, 40.0)
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Connections:
- CAN0 pad 1: CAN1 -> unconnected-(CAN0-Pin_1-Pad1)
- CAN0 pad 3: CAN3 -> CAN1
- CAN0 pad 4: CAN4 -> unconnected-(CAN0-Pin_4-Pad4)
Routing:
- net OUT_3_3_V: track 0.00 -> 304.6 mm, vias 0 -> 1
- net BUTTON_5: track 0.00 -> 214.2 mm, vias 0 -> 1
- net BUTTON_4: track 0.00 -> 212.3 mm, vias 0 -> 1
- net +5V: track 0.00 -> 190.2 mm
- net BUTTON_3: track 0.00 -> 159.8 mm, vias 0 -> 1
- net BUTTON_2: track 0.00 -> 154.7 mm, vias 0 -> 1
- net BUTTON_1: track 0.00 -> 147.6 mm, vias 0 -> 1
- net GND: track 0.00 -> 128.8 mm, vias 4 -> 7
- net Net-(AMS0-K): track 0.00 -> 101.3 mm, vias 0 -> 1
- net FUSE_LED: track 0.00 -> 98.4 mm, vias 0 -> 2
- net SAFETY_LED: track 0.00 -> 92.1 mm, vias 0 -> 2
- net PH5: track 0.00 -> 83.1 mm
- net Net-(Q5-D): track 0.00 -> 82.0 mm, vias 0 -> 1
- net PH4: track 0.00 -> 79.2 mm
- net AMS: track 0.00 -> 78.7 mm, vias 0 -> 1
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- added copper zone on B.Cu, net GND
- added copper zone on F.Cu, net GND
- added copper zone on B.Cu, net POWER1
- added copper zone on F.Cu, net POWER1
Other:
- board text added: ".."

Commit message: gotowe
Connections:
- C2 pad 1: +5V -> OUT_5_V
- J1pin200000 pad 1: +5V -> 5V
- J1pin200000 pad 2: OUT_3_3_V -> VCC
- J1pin200000 pad 3: +5V -> 5V
- J1pin200000 pad 4: OUT_3_3_V -> VCC
- J2SO2 pad 1: +5V -> 5V
- J2SO2 pad 2: OUT_3_3_V -> VCC
- J2SO2 pad 3: +5V -> 5V
- J2SO2 pad 4: OUT_3_3_V -> VCC
- R14 pad 1: +5V -> OUT_5_V
- R17 pad 1: +5V -> OUT_5_V
- R9 pad 1: +5V -> OUT_5_V
- U1 pad 5: +5V -> OUT_5_V
- U2 pad 1: +5V -> OUT_5_V
- U2 pad 3: +5V -> OUT_5_V
Routing:
- net +5V: track 190.2 -> 0.00 mm
- net OUT_5_V: track 0.00 -> 169.2 mm
- net OUT_3_3_V: track 304.6 -> 281.3 mm
- net VCC: track 0.00 -> 23.3 mm
- net 5V: track 0.00 -> 21.1 mm
Other:
- board size 200 x 150 mm -> 157.4 x 101.4 mm
- board text added: "RADOSŁAW BARYŁKO DASHBOARD_TESTBOARD"
Changed lines of the file:
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@@
 	(net 7 "P10")
 	(net 8 "PB1")
-	(net 9 "+5V")
+	(net 9 "OUT_5_V")
 	(net 10 "PG3")
 	(net 11 "AMS")
@@
 	(net 70 "Net-(Q5-D)")
 	(net 71 "Net-(SAFETY_LED0-A)")
+	(net 72 "VCC")
+	(net 73 "5V")
 	(footprint "Resistor_SMD:R_0603_1608Metric"
 		(layer "F.Cu")
@@
 			(layers "F.Cu" "F.Mask" "F.Paste")
 			(roundrect_rratio 0.222222)
-			(net 9 "+5V")
+			(net 9 "OUT_5_V")
 			(pintype "passive")
 		)
@@
 			(layers "F.Cu" "F.Mask" "F.Paste")
 			(roundrect_rratio 0.25)
-			(net 9 "+5V")
+			(net 9 "OUT_5_V")
 			(pinfunction "IN")
 			(pintype "power_in")
@@
 			(layers "F.Cu" "F.Mask" "F.Paste")
 			(roundrect_rratio 0.25)
-			(net 9 "+5V")
+			(net 9 "OUT_5_V")
 			(pinfunction "EN")
 			(pintype "input")
@@
 			(layers "F.Cu" "F.Mask" "F.Paste")
 			(roundrect_rratio 0.222222)
-			(net 9 "+5V")
+			(net 9 "OUT_5_V")
 			(pintype "passive")
 		)
@@
 			(layers "*.Cu" "*.Mask")
 			(remove_unused_layers no)
-			(net 9 "+5V")
+			(net 73 "5V")
 			(pinfunction "Pin_1")
 			(pintype "passive")
@@
 			(layers "*.Cu" "*.Mask")
 			(remove_unused_layers no)
-			(net 46 "OUT_3_3_V")
+			(net 72 "VCC")
 			(pinfunction "Pin_2")
 			(pintype "passive")
@@
 			(layers "*.Cu" "*.Mask")
 			(remove_unused_layers no)
-			(net 9 "+5V")
+			(net 73 "5V")
 			(pinfunction "Pin_3")
 			(pintype "passive")
@@
 			(layers "*.Cu" "*.Mask")
 			(remove_unused_layers no)
-			(net 46 "OUT_3_3_V")
+			(net 72 "VCC")
 			(pinfunction "Pin_4")
 			(pintype "passive")
@@
 			(layers "F.Cu" "F.Mask" "F.Paste")
 			(roundrect_rratio 0.25)
-			(net 9 "+5V")
+			(net 9 "OUT_5_V")
 			(pintype "passive")
 		)
@@
 			(layers "F.Cu" "F.Mask" "F.Paste")
 			(roundrect_rratio 0.222222)
-			(net 9 "+5V")
+			(net 9 "OUT_5_V")
 			(pintype "passive")
 		)
@@
 			(layers "F.Cu" "F.Mask" "F.Paste")
 			(roundrect_rratio 0.25)
-			(net 9 "+5V")
+			(net 9 "OUT_5_V")
 			(pinfunction "OUT")
 			(pintype "power_out")
@@
 			(layers "*.Cu" "*.Mask")
 			(remove_unused_layers no)
-			(net 9 "+5V")
+			(net 73 "5V")
 			(pinfunction "Pin_1")
 			(pintype "passive")
@@
 			(layers "*.Cu" "*.Mask")
 			(remove_unused_layers no)
-			(net 46 "OUT_3_3_V")
+			(net 72 "VCC")
 			(pinfunction "Pin_2")
 			(pintype "passive")
@@
 			(layers "*.Cu" "*.Mask")
 			(remove_unused_layers no)
-			(net 9 "+5V")
+			(net 73 "5V")
 			(pinfunction "Pin_3")
 			(pintype "passive")
@@
 			(layers "*.Cu" "*.Mask")
 			(remove_unused_layers no)
-			(net 46 "OUT_3_3_V")
+			(net 72 "VCC")
 			(pinfunction "Pin_4")
 			(pintype "passive")
@@
 	)
 	(gr_rect
-		(start 47.5 23.5)
-		(end 247.5 173.5)
+		(start 90.1 23.5)
+		(end 247.5 124.9)
 		(stroke
 			(width 0.05)
@@
 		(layer "Edge.Cuts")
 	)
+	(gr_text "RADOSŁAW BARYŁKO\nDASHBOARD_TESTBOARD"
+		(at 242.5 122.1 0)
+		(layer "B.SilkS")
+		(effects
+			(font
+				(size 1 1)
+				(thickness 0.1)
+			)
+			(justify left bottom mirror)
+		)
+	)
 	(gr_text ".."
 		(at 125.8 56.8 0)
@@
 	)
 	(segment
-		(start 223.65 37.07)
-		(end 222.38 37.07)
-		(width 0.2)
-		(layer "F.Cu")
-		(net 9)
-	)
-	(segment
 		(start 111.601 26.999)
 		(end 112.890364 26.999)
@@
 	)
 	(segment
-		(start 223.63 37.09)
-		(end 223.65 37.07)
-		(width 0.2)
-		(layer "F.Cu")
-		(net 9)
-	)
-	(segment
 		(start 212.025 106.575)
 		(end 204.675 106.575)
@@
 	)
 	(segment
-		(start 223.63 55.6)
-		(end 223.63 37.09)
-		(width 0.2)
-		(layer "F.Cu")
-		(net 9)
-	)
-	(segment
 		(start 114.9 29.008636)
 		(end 114.9 49.850058)
@@
 	)
 	(segment
-		(start 223.63 55.6)
-		(end 223.63 56.87)
-		(width 0.2)
-		(layer "F.Cu")
-		(net 9)
-	)
-	(segment
 		(start 214.359 38.2)
 		(end 213.35 38.2)
@@
 	)
 	(segment
-		(start 223.65 35.8)
-		(end 222.38 35.8)
-		(width 0.2)
-		(layer "F.Cu")
-		(net 46)
-	)
-	(segment
 		(start 149.3125 106.4)
 		(end 137.3125 94.4)
@@
 	)
 	(segment
-		(start 224.9 55.6)
-		(end 224.9 36.342894)
-		(width 0.2)
-		(layer "F.Cu")
-		(net 46)
-	)
-	(segment
 		(start 163.3125 106.4)
 		(end 150.5125 93.6)
@@
 	)
 	(segment
-		(start 224.357106 35.8)
-		(end 223.65 35.8)
-		(width 0.2)
-		(layer "F.Cu")
-		(net 46)
-	)
-	(segment
 		(start 202.225 106.4)
 		(end 202.225 108.325)
@@
 	)
 	(segment
-		(start 224.9 36.342894)
-		(end 224.357106 35.8)
-		(width 0.2)
-		(layer "F.Cu")
-		(net 46)
-	)
-	(segment
 		(start 202.225 106.4)
 		(end 175.5 106.4)
@@
 	)
 	(segment
-		(start 224.9 56.87)
-		(end 224.9 55.6)
-		(width 0.2)
-		(layer "F.Cu")
-		(net 46)
-	)
-	(segment
 		(start 175.5 106.4)
 		(end 162.9 93.8)
@@
 		(net 71)
 	)
+	(segment
+		(start 223.65 35.8)
+		(end 222.38 35.8)
+		(width 0.2)
+		(layer "F.Cu")
+		(net 72)
+	)
+	(segment
+		(start 224.9 55.6)
+		(end 224.9 36.342894)
+		(width 0.2)
+		(layer "F.Cu")
+		(net 72)
+	)
+	(segment
+		(start 224.357106 35.8)
+		(end 223.65 35.8)
+		(width 0.2)
+		(layer "F.Cu")
+		(net 72)
+	)
+	(segment
+		(start 224.9 36.342894)
+		(end 224.357106 35.8)
+		(width 0.2)
+		(layer "F.Cu")
+		(net 72)
+	)
+	(segment
+		(start 224.9 56.87)
+		(end 224.9 55.6)
+		(width 0.2)
+		(layer "F.Cu")
+		(net 72)
+	)
+	(segment
+		(start 223.65 37.07)
+		(end 222.38 37.07)
+		(width 0.2)
+		(layer "F.Cu")
+		(net 73)
+	)
+	(segment
+		(start 223.63 37.09)
+		(end 223.65 37.07)
+		(width 0.2)
+		(layer "F.Cu")
+		(net 73)
+	)
+	(segment
+		(start 223.63 55.6)
+		(end 223.63 37.09)
+		(width 0.2)
+		(layer "F.Cu")
+		(net 73)
+	)
+	(segment
+		(start 223.63 55.6)
+		(end 223.63 56.87)
+		(width 0.2)
+		(layer "F.Cu")
+		(net 73)
+	)
 	(zone
 		(net 5)
@@
 		(polygon
 			(pts
-				(xy 63.6 27.9) (xy 65.2 153.5) (xy 245.1 153.9) (xy 245.9 24.3)
+				(xy 90.4 23.9) (xy 91.106537 124.213136) (xy 247.4 124.8) (xy 247.2 23.9)
 			)
 		)

Commit message: jest jako tako
Parts:
- removed TERM_0: Conn_01x02_Pin, Connector_PinHeader_1.27mm:PinHeader_1x02_P1.27mm_Vertical
- added D8: PESD2CAN.215, Package_TO_SOT_SMD:SOT-23-3, F.Cu at (149.1, 33.5)
- CAN0: footprint Connector_Dsub:DSUB-9_Pins_Horizontal_P2.77x2.84mm_EdgePinOffset4.94mm_Housed_MountingHolesOffset4.94mm -> Connector_Dsub:DSUB-9_Socket_Vertical_P2.77x2.84mm
- CAN1: moved to B.Cu
- SW1, SW2, SW3, SW4, SW5: footprint Button_Switch_SMD:SW_Push_1TS009xxxx-xxxx-xxxx_6x6x5mm -> Button_Switch_SMD:SW_Push_1P1T_NO_E-Switch_TL3301NxxxxxG
- moved USR_BTN1 136.8 mm to (100.5, 109.4), turned to 90 degrees
- moved DRS_BTN1 125.1 mm to (100.4, 93.0), turned to 90 degrees
- moved J1 119.0 mm to (102.7, 30.7)
- moved TSA_BTN1 105.2 mm to (100.5, 77.3), turned to 90 degrees
- moved CS_BTN1 104.6 mm to (100.8, 44.2), turned to 90 degrees
- moved R1 104.5 mm to (98.7, 51.9)
- moved RTD_BTN1 103.5 mm to (100.7, 60.7), turned to 90 degrees
- moved R4 100.6 mm to (98.5, 117.2)
- moved R2 99.5 mm to (98.5, 67.1)
- moved R3 97.1 mm to (98.3, 85.2)
- moved J2 96.3 mm to (108.1, 30.7), turned to 180 degrees
- moved R5 91.2 mm to (98.5, 101.0)
- moved J3 87.6 mm to (113.6, 30.6), turned to 180 degrees
- moved SW4 58.0 mm to (98.5, 117.2), turned to -90 degrees
- moved SW3 51.5 mm to (98.3, 85.2), turned to -90 degrees
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- renumbered AMS1 to J1, SAFETY_LED1 to J2, FUSE_LED1 to J3
Connections:
- net 5V renamed /SOCKETS_2X20/<NO NET>
- net AMS renamed /LED_1
- net BUTTON_1 renamed /BUTTON_1
- net BUTTON_2 renamed /BUTTON_2
- net BUTTON_3 renamed /BUTTON_3
- net BUTTON_4 renamed /BUTTON_4
- net BUTTON_5 renamed /BUTTON_5
- net CAN1 renamed /CAN/CAN_GND
- net CAN3 renamed /CAN/CAN_P
- net CAN4 renamed /CAN/CAN_VDD
- net FUSE_LED renamed /LED_2
- net OUT_3_3_V renamed +3.3V
- net OUT_5_V renamed +5V
- net P10 renamed /SOCKETS_2X20/P10
- net P14 renamed /SOCKETS_2X20/P14
- net P15 renamed /SOCKETS_2X20/P15
- net PA10 renamed /SOCKETS_2X20/PA10
- net PA11 renamed /SOCKETS_2X20/PA11
- net PA12 renamed /SOCKETS_2X20/PA12
- net PA15 renamed /SOCKETS_2X20/PA15
- net PA3 renamed /SOCKETS_2X20/PA3
- net PA4 renamed /SOCKETS_2X20/PA4
- net PA5 renamed /SOCKETS_2X20/PA5
- net PA6 renamed /SOCKETS_2X20/PA6
- net PA7 renamed /SOCKETS_2X20/PA7
- net PA8 renamed /SOCKETS_2X20/PA8
- net PB0 renamed /SOCKETS_2X20/PB0
- net PB1 renamed /SOCKETS_2X20/PB1
- net PB10 renamed /SOCKETS_2X20/PB10
- net PB15 renamed /SOCKETS_2X20/PB15
- net PB2 renamed /SOCKETS_2X20/PB2
- net PB5 renamed /SOCKETS_2X20/PB5
- net PB6 renamed /SOCKETS_2X20/PB6
- net PB7 renamed /SOCKETS_2X20/PB7
- net PC7 renamed /SOCKETS_2X20/PC7
- net PE40 renamed /SOCKETS_2X20/PE40
- net PG10 renamed /SOCKETS_2X20/PG10
- net PG2 renamed /SOCKETS_2X20/PG2
- net PG3 renamed /SOCKETS_2X20/PG3
- net PG4 renamed /SOCKETS_2X20/PG4
- net PG9 renamed /SOCKETS_2X20/PG9
- net PH11 renamed /SOCKETS_2X20/PH11
- net PH4 renamed /SOCKETS_2X20/PH4
- net PH5 renamed /SOCKETS_2X20/PH5
- net POWER1 renamed /POWER/POWER1
- net POWER_EN renamed /POWER/POWER_EN
- net SAFETY_LED renamed /LED_3
- net SWD1 renamed /SWD/SWD_VCC_+3.3V
- net SWD2 renamed /SWD/SWD_SW_CLK
- net SWD4 renamed /SWD/SWD_SW_DIO
- net SWD5 renamed /SWD/SWD_RST
- net SWD6 renamed /SWD/SWD_SWO
- net VCC renamed /SOCKETS_2X20/VCC
- ALT_CAN0 pad 1: CAN2 -> /CAN/CAN_N
- CAN0 pad 2: CAN2 -> /CAN/CAN_N
- CAN1 pad 2: CAN2 -> /CAN/CAN_N
- R11 pad 1: Net-(TERM_0-Pin_2) -> /CAN/CAN_N
- SWD0 pad 3: SWD3 -> GND
- SWD1 pad 3: SWD3 -> GND
- SWD2 pad 3: SWD3 -> GND
Routing:
- net /BUTTON_5: track 214.2 -> 20.1 mm, vias 1 -> 0
- net /BUTTON_4: track 212.3 -> 19.7 mm, vias 1 -> 0
- net /SOCKETS_2X20/PH11: track 65.2 -> 217.5 mm
- net /SOCKETS_2X20/PA5: track 26.0 -> 168.1 mm, vias 0 -> 2
- net /BUTTON_3: track 159.8 -> 19.8 mm, vias 1 -> 0
- net /BUTTON_2: track 154.7 -> 18.3 mm, vias 1 -> 0
- net /SOCKETS_2X20/PB0: track 50.6 -> 186.5 mm
- net /SOCKETS_2X20/PA3: track 68.6 -> 204.2 mm
- net /SOCKETS_2X20/P14: track 49.1 -> 178.8 mm
- net /BUTTON_1: track 147.6 -> 19.5 mm, vias 1 -> 0
- net /SOCKETS_2X20/PA15: track 52.6 -> 176.6 mm
- net /SOCKETS_2X20/PH5: track 83.1 -> 173.7 mm
- net /SOCKETS_2X20/PH4: track 79.2 -> 162.5 mm
- net /CAN/CAN_N: track 0.00 -> 67.6 mm
- net CAN2: track 60.3 -> 0.00 mm
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Other:
- board size 157.4 x 101.4 mm -> 157.4 x 98.9 mm

Commit message: jest lepiej
Parts:
- removed SWD1: Conn_01x06_MountingPin, Connector_PinHeader_1.27mm:PinHeader_1x06_P1.27mm_Vertical
- SWD0: value Conn_01x06_MountingPin -> Conn_02x05_Odd_Even; footprint Connector_Molex:Molex_CLIK-Mate_502382-0670_1x06-1MP_P1.25mm_Vertical -> Connector_IDC:IDC-Header_2x05_P2.54mm_Vertical
- SWD2: moved to B.Cu
- moved SWD2 25.1 mm to (175.1, 64.4), turned to 0 degrees
- moved SWD0 10.3 mm to (178.5, 38.1), turned to -90 degrees
Connections:
- SWD0 pad 2: /SWD/SWD_SW_CLK -> /SWD/SWD_SW_DIO
- SWD0 pad 4: /SWD/SWD_SW_DIO -> /SWD/SWD_SW_CLK
- SWD0 pad 5: /SWD/SWD_RST -> GND
Routing:
- net /SWD/SWD_VCC_+3.3V: track 45.6 -> 27.7 mm
- net GND: track 163.3 -> 175.1 mm, vias 7 -> 11
- net /SWD/SWD_SW_CLK: track 43.2 -> 31.6 mm
- net /SWD/SWD_RST: track 31.9 -> 25.1 mm
- net /SWD/SWD_SW_DIO: track 36.1 -> 31.2 mm
- net /SWD/SWD_SWO: track 28.2 -> 31.7 mm

Commit message: jest
Parts:
- removed J4POWER0: Conn_01x06_MountingPin, Connector_Molex:Molex_CLIK-Mate_502382-0670_1x06-1MP_P1.25mm_Vertical
- removed SWD0: Conn_02x05_Odd_Even, Connector_IDC:IDC-Header_2x05_P2.54mm_Vertical
- added J6: Conn_02x10_Odd_Even, Connector_IDC:IDC-Header_2x10_P2.54mm_Vertical, B.Cu at (169.5, 37.1)
Connections:
- J5POWER1 pad 4: /POWER/POWER_EN -> unconnected-(J5POWER1-Pin_4-Pad4)
Routing:
- net /POWER/POWER_EN: track 72.8 -> 0.00 mm
- net GND: track 175.1 -> 149.8 mm, vias 11 -> 10
- net /SWD/SWD_SW_DIO: track 31.2 -> 39.4 mm
- net /SWD/SWD_RST: track 25.1 -> 29.2 mm
- net /SWD/SWD_SW_CLK: track 31.6 -> 28.7 mm
- net /SWD/SWD_SWO: track 31.7 -> 34.6 mm
- net /SWD/SWD_VCC_+3.3V: track 27.7 -> 29.7 mm

Commit message: gotowe
Parts:
- added J4: Conn_01x01, footprints:PJ3253, B.Cu at (237.4, 39.8)
- added J5: Conn_01x01, footprints:PJ3253, B.Cu at (251.3, 47.3)
Routing:
- net GND: track 149.8 -> 131.8 mm, vias 10 -> 11
- net /SOCKETS_2X20/PA5: track 168.1 -> 168.0 mm, vias 2 -> 0
Other:
- board size 157.4 x 98.9 mm -> 170.5 x 98.9 mm

Commit message: g
Parts:
- moved CAN1 0.10 mm to (125.0, 54.3)
Routing:
- net GND: track 131.8 -> 67.3 mm, vias 11 -> 12
- net /SOCKETS_2X20/<NO NET>: track 21.1 -> 41.4 mm
- net /SOCKETS_2X20/PA8: track 71.7 -> 89.0 mm
- net /SOCKETS_2X20/PB0: track 186.5 -> 200.5 mm
- net /SOCKETS_2X20/PA5: track 168.0 -> 156.1 mm
- net /SOCKETS_2X20/PA3: track 204.2 -> 214.7 mm
- net /SOCKETS_2X20/PB2: track 68.1 -> 77.4 mm
- net /CAN/CAN_GND: track 29.6 -> 38.5 mm
- net /SOCKETS_2X20/P14: track 178.8 -> 187.3 mm
- net /SOCKETS_2X20/PH5: track 173.7 -> 181.5 mm
- net /SOCKETS_2X20/PA6: track 53.8 -> 61.4 mm
- net /SOCKETS_2X20/PA7: track 50.2 -> 56.9 mm
- net /SOCKETS_2X20/P10: track 44.2 -> 50.0 mm
- net /SOCKETS_2X20/PC7: track 40.6 -> 45.5 mm
- net +5V: track 187.3 -> 191.7 mm
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
Commit message: g2
Parts:
- removed J6: Conn_02x10_Odd_Even, Connector_IDC:IDC-Header_2x10_P2.54mm_Vertical
- added J7: FTSH, footprints:FTSH-107-XX-YYY-DV-K-A, B.Cu at (179.1, 41.4)
- added J8: Conn_01x03_Socket, Connector_BarrelJack:BarrelJack_Kycon_KLDX-0202-xC_Horizontal, F.Cu at (246.2, 54.0)
- D8, R11: moved to B.Cu
- moved R11 8.98 mm to (160.0, 40.2)
- moved J5 4.91 mm to (251.6, 42.4)
- moved TERM_1 3.69 mm to (157.1, 41.0), turned to 0 degrees
- moved J4 3.28 mm to (235.4, 42.4)
- moved D8 1.57 mm to (150.7, 33.6), turned to 0 degrees
Connections:
- SWD2 pad 6: /SWD/SWD_SWO -> unconnected-(SWD2-Pin_6-Pad6)
Routing:
- net /SWD/SWD_SWO: track 34.6 -> 0.00 mm
- net GND: track 67.3 -> 41.6 mm, vias 12 -> 13
- net /CAN/CAN_N: track 71.3 -> 61.4 mm
- net /SWD/SWD_SW_DIO: track 39.4 -> 31.0 mm
- net /SWD/SWD_SW_CLK: track 28.7 -> 21.7 mm
- net /SWD/SWD_RST: track 29.2 -> 24.2 mm
- net Net-(TERM_1-Pin_1): track 7.57 -> 3.19 mm
- net /CAN/CAN_P: track 58.7 -> 57.2 mm
- net /SWD/SWD_VCC_+3.3V: track 29.7 -> 30.8 mm
- net /POWER/POWER1: vias 2 -> 0
Other:
- board size 170.5 x 98.9 mm -> 175.1 x 98.9 mm
