File: hardware/PUTM_EV_DASHBOARD_SOCKET_2025/SWD.kicad_sch (KiCad schematic)
At the start: 3 parts

Commit message: prawie gotowe
Parts:
- SWD0: footprint Connector_Dsub:DSUB-9_Pins_Horizontal_P2.77x2.54mm_EdgePinOffset9.40mm -> Connector_Molex:Molex_CLIK-Mate_502382-0670_1x06-1MP_P1.25mm_Vertical
- SWD2: footprint Connector_PinHeader_1.27mm:PinHeader_1x06_P1.27mm_Vertical -> Connector_Wire:SolderWire-0.1sqmm_1x06_P3.6mm_D0.4mm_OD1mm_Relief
Changed lines of the file:
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@@
 			)
 		)
-		(property "Footprint" "Connector_Dsub:DSUB-9_Pins_Horizontal_P2.77x2.54mm_EdgePinOffset9.40mm"
+		(property "Footprint" "Connector_Molex:Molex_CLIK-Mate_502382-0670_1x06-1MP_P1.25mm_Vertical"
 			(at 95.25 78.74 0)
 			(effects
@@
 			)
 		)
-		(property "Footprint" "Connector_PinHeader_1.27mm:PinHeader_1x06_P1.27mm_Vertical"
+		(property "Footprint" "Connector_Wire:SolderWire-0.1sqmm_1x06_P3.6mm_D0.4mm_OD1mm_Relief"
 			(at 193.04 80.01 0)
 			(effects

Commit message: jest jako tako
Connections:
- net SWD1 renamed SWD_VCC_+3.3V
- net SWD2 renamed SWD_SW_CLK
- net SWD3 renamed GND
- net SWD4 renamed SWD_SW_DIO
- net SWD5 renamed SWD_RST
- net SWD6 renamed SWD_SWO

Commit message: jest lepiej
Parts:
- removed SWD0: Conn_01x06_MountingPin, Connector_Molex:Molex_CLIK-Mate_502382-0670_1x06-1MP_P1.25mm_Vertical, symbol Connector_Generic_MountingPin:Conn_01x06_MountingPin
- removed SWD1: Conn_01x06_MountingPin, Connector_PinHeader_1.27mm:PinHeader_1x06_P1.27mm_Vertical, symbol Connector_Generic_MountingPin:Conn_01x06_MountingPin
- added SWD0: Conn_02x05_Odd_Even, Connector_IDC:IDC-Header_2x05_P2.54mm_Vertical, symbol Connector_Generic:Conn_02x05_Odd_Even
Connections:
- net GND: now also SWD0.3 (Pin_3), SWD0.5 (Pin_5), SWD0.9 (Pin_9)
- net SWD_RST: now also SWD0.10 (Pin_10)
- net SWD_SWO: now also SWD0.6 (Pin_6)
- net SWD_SW_CLK: now also SWD0.4 (Pin_4)
- net SWD_SW_DIO: now also SWD0.2 (Pin_2)
- net SWD_VCC_+3.3V: now also SWD0.1 (Pin_1)
- no-connect marks 0 -> 2

Commit message: jest
Parts:
- removed SWD0: Conn_02x05_Odd_Even, Connector_IDC:IDC-Header_2x05_P2.54mm_Vertical, symbol Connector_Generic:Conn_02x05_Odd_Even
- added J6: Conn_02x10_Odd_Even, Connector_IDC:IDC-Header_2x10_P2.54mm_Vertical, symbol Connector_Generic:Conn_02x10_Odd_Even
Connections:
- net GND: now also J6.10 (Pin_10), J6.12 (Pin_12), J6.14 (Pin_14), J6.16 (Pin_16), J6.18 (Pin_18), J6.20 (Pin_20), J6.3 (Pin_3), J6.4 (Pin_4), J6.5 (Pin_5), J6.6 (Pin_6), J6.8 (Pin_8)
- net SWD_RST: now also J6.15 (Pin_15)
- net SWD_SWO: now also J6.13 (Pin_13)
- net SWD_SW_CLK: now also J6.9 (Pin_9)
- net SWD_SW_DIO: now also J6.7 (Pin_7)
- net SWD_VCC_+3.3V: now also J6.1 (Pin_1), J6.2 (Pin_2)
- no-connect marks 2 -> 3

Commit message: g2
Parts:
- removed J6: Conn_02x10_Odd_Even, Connector_IDC:IDC-Header_2x10_P2.54mm_Vertical, symbol Connector_Generic:Conn_02x10_Odd_Even
- added J7: FTSH, footprints:FTSH-107-XX-YYY-DV-K-A, symbol ftsh-107-01-l-dv-k-a:FTSH-107-01-L-DV-K-A
Connections:
- net GND: now also J7.11 (Pin_11), J7.5 (Pin_5), J7.7 (Pin_7)
- net SWD_RST: now also J7.12 (Pin_12)
- net SWD_SW_CLK: now also J7.6 (Pin_6)
- net SWD_SW_DIO: now also J7.4 (Pin_4)
- net SWD_VCC_+3.3V: now also J7.3 (Pin_3)
- net SWD_SWO: no longer names the net of SWD2.6 (Pin_6)
- no-connect marks 3 -> 8

Commit message: g3
Other:
- note added: "ZŁĄCZA SWD"
- moved on the sheet: SWD2
Changed lines of the file:
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@@
 	(generator_version "9.0")
 	(paper "A4")
+	(rectangle
+		(start 76.2 64.77)
+		(end 198.755 106.045)
+		(stroke
+			(width 0)
+			(type default)
+		)
+		(fill
+			(type none)
+		)
+	)
+	(text "ZŁĄCZA SWD\n"
+		(exclude_from_sim no)
+		(at 121.666 71.628 0)
+		(effects
+			(font
+				(size 1.27 1.27)
+			)
+		)
+	)
 	(junction
 		(at 97.79 91.44)
@@
 	)
 	(no_connect
-		(at 187.96 87.63)
+		(at 162.56 93.98)
 	)
 	(wire
@@
 	(wire
 		(pts
-			(xy 180.34 77.47) (xy 187.96 77.47)
+			(xy 154.94 83.82) (xy 162.56 83.82)
 		)
 		(stroke
@@
 	(wire
 		(pts
-			(xy 180.34 82.55) (xy 187.96 82.55)
+			(xy 154.94 88.9) (xy 162.56 88.9)
 		)
 		(stroke
@@
 	(hierarchical_label "SWD_SW_CLK"
 		(shape input)
-		(at 180.34 77.47 180)
+		(at 154.94 83.82 180)
 		(effects
 			(font
@@
 	(hierarchical_label "SWD_VCC_+3.3V"
 		(shape input)
-		(at 187.96 74.93 180)
+		(at 162.56 81.28 180)
 		(effects
 			(font
@@
 	(hierarchical_label "SWD_SW_DIO"
 		(shape input)
-		(at 180.34 82.55 180)
+		(at 154.94 88.9 180)
 		(effects
 			(font
@@
 	(hierarchical_label "SWD_RST"
 		(shape input)
-		(at 187.96 85.09 180)
+		(at 162.56 91.44 180)
 		(effects
 			(font
@@
 	(symbol
 		(lib_id "power:GND")
-		(at 187.96 80.01 270)
+		(at 162.56 86.36 270)
 		(unit 1)
 		(exclude_from_sim no)
@@
 		(fields_autoplaced yes)
 		(property "Reference" "#PWR042"
-			(at 181.61 80.01 0)
+			(at 156.21 86.36 0)
 			(effects
 				(font
@@
 		)
 		(property "Value" "GND"
-			(at 184.15 80.0099 90)
+			(at 158.75 86.3599 90)
 			(effects
 				(font
@@
 		)
 		(property "Footprint" ""
-			(at 187.96 80.01 0)
+			(at 162.56 86.36 0)
 			(effects
 				(font
@@
 		)
 		(property "Datasheet" ""
-			(at 187.96 80.01 0)
+			(at 162.56 86.36 0)
 			(effects
 				(font
@@
 		)
 		(property "Description" "Power symbol creates a global label with name \"GND\" , ground"
-			(at 187.96 80.01 0)
+			(at 162.56 86.36 0)
 			(effects
 				(font
@@
 	(symbol
 		(lib_id "Connector_Generic_MountingPin:Conn_01x06_MountingPin")
-		(at 193.04 80.01 0)
+		(at 167.64 86.36 0)
 		(unit 1)
 		(exclude_from_sim no)
@@
 		(fields_autoplaced yes)
 		(property "Reference" "SWD2"
-			(at 195.58 80.0099 0)
+			(at 170.18 86.3599 0)
 			(effects
 				(font
@@
 		)
 		(property "Value" "Conn_01x06_MountingPin"
-			(at 195.58 82.5499 0)
+			(at 170.18 88.8999 0)
 			(effects
 				(font
@@
 		)
 		(property "Footprint" "Connector_Wire:SolderWire-0.1sqmm_1x06_P3.6mm_D0.4mm_OD1mm_Relief"
-			(at 193.04 80.01 0)
+			(at 167.64 86.36 0)
 			(effects
 				(font
@@
 		)
 		(property "Datasheet" "~"
-			(at 193.04 80.01 0)
+			(at 167.64 86.36 0)
 			(effects
 				(font
@@
 		)
 		(property "Description" "Generic connectable mounting pin connector, single row, 01x06, script generated (kicad-library-utils/schlib/autogen/connector/)"
-			(at 193.04 80.01 0)
-			(effects
-				(font
+			(at 167.64 86.36 0)
+			(effects
+				(font

Commit message: poprawione opisy i złącze swd
Connections:
- net GND: no longer SWD2.3 (Pin_3)
- net SWD_SWO: now reaches J7.8 (Pin_8)
- net SWD_SWO: now also SWD2.3 (Pin_3)
- no-connect marks 8 -> 7
Changed lines of the file:
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@@
-	)
-	(no_connect
-		(at 113.03 86.36)
 	)
 	(no_connect
@@
 			(width 0)
 			(type default)
+		)
+	)
+	(global_label "SWD_SWO"
+		(shape input)
+		(at 113.03 86.36 0)
+		(fields_autoplaced yes)
+		(effects
+			(font
+				(size 1.27 1.27)
+			)
+			(justify left)
+		)
+		(property "Intersheetrefs" "${INTERSHEET_REFS}"
+			(at 124.9051 86.36 0)
+			(effects
+				(font
+					(size 1.27 1.27)
+				)
+				(justify left)
+				(hide yes)
+			)
+		)
+	)
+	(global_label "SWD_SWO"
+		(shape input)
+		(at 162.56 86.36 180)
+		(fields_autoplaced yes)
+		(effects
+			(font
+				(size 1.27 1.27)
+			)
+			(justify right)
+		)
+		(property "Intersheetrefs" "${INTERSHEET_REFS}"
+			(at 150.6849 86.36 0)
+			(effects
+				(font
+					(size 1.27 1.27)
+				)
+				(justify right)
+				(hide yes)
+			)
 		)
 	)
@@
 					(unit 1)
 				)
-			)
-		)
-	)
-	(symbol
-		(lib_id "power:GND")
-		(at 162.56 86.36 270)
-		(unit 1)
-		(exclude_from_sim no)
-		(in_bom yes)
-		(on_board yes)
-		(dnp no)
-		(fields_autoplaced yes)
-		(property "Reference" "#PWR042"
-			(at 156.21 86.36 0)
-			(effects
-				(font
-					(size 1.27 1.27)
-				)
-				(hide yes)
-			)
-		)
-		(property "Value" "GND"
-			(at 158.75 86.3599 90)
-			(effects
-				(font
-					(size 1.27 1.27)
-				)
-				(justify right)
-			)
-		)
-		(property "Footprint" ""
-			(at 162.56 86.36 0)
-			(effects
-				(font
-					(size 1.27 1.27)
-				)
-				(hide yes)
-			)
-		)
-		(property "Datasheet" ""
-			(at 162.56 86.36 0)
-			(effects
-				(font
-					(size 1.27 1.27)
-				)
-				(hide yes)
-			)
-		)
-		(property "Description" "Power symbol creates a global label with name \"GND\" , ground"
-			(at 162.56 86.36 0)
-			(effects
-				(font
-					(size 1.27 1.27)
-				)
-				(hide yes)
-			)
-		)
-		(pin "1"
-		)
-		(instances
-			(project "PUTM_EV_DASHBOARD_SOCKET_2025"
-				(path "/8dcb9295-4fa2-433e-bd2f-4b006d008a4e/9b1bc52f-6033-4f71-8f99-a4060d1be2be"
-					(reference "#PWR042")
-					(unit 1)
-				)

Commit message: poprawione opisy i złącze swd, gnazdo POWER jest na krawędzi płytki
Changed lines of the file:
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@@
-		)
-	)
-	(global_label "SWD_SWO"
-		(shape input)
-		(at 113.03 86.36 0)
-		(fields_autoplaced yes)
-		(effects
-			(font
-				(size 1.27 1.27)
-			)
-			(justify left)
-		)
-		(property "Intersheetrefs" "${INTERSHEET_REFS}"
-			(at 124.9051 86.36 0)
-			(effects
-				(font
-					(size 1.27 1.27)
-				)
-				(justify left)
-				(hide yes)
-			)
-		)
-	)
-	(global_label "SWD_SWO"
-		(shape input)
-		(at 162.56 86.36 180)
-		(fields_autoplaced yes)
-		(effects
-			(font
-				(size 1.27 1.27)
-			)
-			(justify right)
-		)
-		(property "Intersheetrefs" "${INTERSHEET_REFS}"
-			(at 150.6849 86.36 0)
-			(effects
-				(font
-					(size 1.27 1.27)
-				)
-				(justify right)
-				(hide yes)
-			)
 		)
 	)
@@
 			)
 			(justify right)
+		)
+	)
+	(hierarchical_label "SWD_SWO"
+		(shape input)
+		(at 113.03 86.36 0)
+		(effects
+			(font
+				(size 1.27 1.27)
+			)
+			(justify left)
 		)
 	)
@@
 		(effects
 			(font
+				(size 1.27 1.27)
+			)
+			(justify right)
+		)
+	)
+	(hierarchical_label "SWD_SWO"
+		(shape input)
+		(at 162.56 86.36 180)
+		(effects
+			(font
