File: hardware/PUTM_EV_DASHBOARD_SOCKET_2025/SWD.kicad_sch (KiCad schematic)
At the start: 2 parts, among them J7 FTSH

Commit message: Bogracz Czas przygotowania: 3 godziny 30 minut Liczba porcji: 2100 g gulaszu  W 100 g dania: Wartość energetyczna 156 kcal Węglowodany 5 g - W tym cukry 2 g Białko 7 g Tłuszcze 12 g
Składniki

800 g mięsa wołowego - np. pręga oraz łopatka
200 g boczku gotowanego wędzonego
100 g dobrej jakosci słoniny
6 łyżek dobrej jakości smalcu - około 100 g
2 średniej wielkości cebule - około 330 g
2 średniej wielkości czerwone papryki - około 400 g
5 ząbków czosnku - około 25 g
500 g ziemniaków - można pominąć lub dać kluseczki
2 łyżki koncentratu pomidorowego - do 50 g
400 ml wody - trochę więcej niż 1,5 szklanki
zioła i przyprawy: 2 listki laurowe, 3 ziarna ziela angielskiego; 1 pełna łyżeczka słodkiej papryki; 1 płaska łyżeczka soli; po pół łyżeczki wędzonej i ostrej papryki; 1/3 łyżeczki czarnego pieprzu
Składniki:
Bogracz
Szklanka ma u mnie pojemność 250 ml.

Warzywa ważone były przed ewentualnym obraniem/przygotowaniem. Zawsze podaję wagę użytych przeze mnie warzyw lub owoców. Nie trzeba jednak stosować się do wytycznych co do grama. Wagi podawane są po to, by łatwiej Wam było zorientować się, jaka mniej więcej ilość potrzebna jest do zrobienia danego dania.

Kalorie policzone zostały na podstawie użytych przeze mnie składników. Jest to więc orientacyjna liczba kalorii, ponieważ Twoje składniki mogą mieć inną liczbę kalorii niż te, których użyłam ja. Z podanej ilości składników otrzymasz Bogracz o wadze około 2100 gramów. Zanim zaczniesz szykować ten gulasz, polecam najpierw przeczytać cały przepis, by przygotować się odpowiednio wcześniej do kolejnych etapów wykonania.

UWAGA: Bogracz, to rodzaj kociołka stalowego lub emaliowanego, który rozszerza się ku górze. Kociołek podwieszany jest na trójnogu i wieszany na metalowym łańcuchu. Bogracz wisi nad ogniskiem, a w środku gotuje się węgierski gulasz. Zaczęto zatem nazywać tak samo i danie. Ponieważ zdecydowana większość Czytelników nie ma możliwości szykowania tego gulaszu w kociołku na świeżym powietrzu, podaję przepis na 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
Connections:
- net GND: now also SWD2.3 (Pin_3)
- net SWD_SWO: now also SWD2.6 (Pin_6); no longer SWD2.3 (Pin_3)
- no-connect marks 7 -> 6
Changed lines of the file:
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@@
 		(at 113.03 93.98)
 	)
-	(no_connect
-		(at 162.56 93.98)
-	)
 	(wire
 		(pts
@@
 	(hierarchical_label "SWD_SWO"
 		(shape input)
-		(at 162.56 86.36 180)
+		(at 162.56 93.98 180)
 		(effects
 			(font
@@
 		)
 	)
+	(symbol
+		(lib_id "power:GND")
+		(at 162.56 86.36 270)
+		(unit 1)
+		(exclude_from_sim no)
+		(in_bom yes)
+		(on_board yes)
+		(dnp no)
+		(fields_autoplaced yes)
+		(property "Reference" "#PWR045"
+			(at 156.21 86.36 0)
+			(effects
+				(font
+					(size 1.27 1.27)
+				)
+				(hide yes)
+			)
+		)
+		(property "Value" "GND"
+			(at 158.75 86.3599 90)
+			(effects
+				(font
+					(size 1.27 1.27)
+				)
+				(justify right)
+			)
+		)
+		(property "Footprint" ""
+			(at 162.56 86.36 0)
+			(effects
+				(font
+					(size 1.27 1.27)
+				)
+				(hide yes)
+			)
+		)
+		(property "Datasheet" ""
+			(at 162.56 86.36 0)
+			(effects
+				(font
+					(size 1.27 1.27)
+				)
+				(hide yes)
+			)
+		)
+		(property "Description" "Power symbol creates a global label with name \"GND\" , ground"
+			(at 162.56 86.36 0)
+			(effects
+				(font
+					(size 1.27 1.27)
+				)
+				(hide yes)
+			)
+		)
+		(pin "1"
+		)
+		(instances
+			(project "PUTM_EV_DASHBOARD_SOCKET_2025"
+				(path "/8dcb9295-4fa2-433e-bd2f-4b006d008a4e/9b1bc52f-6033-4f71-8f99-a4060d1be2be"
+					(reference "#PWR045")
+					(unit 1)
+				)
+			)
+		)
+	)

Commit message: fixed button text layout
Parts:
- renumbered SWD2 to SWD
Changed lines of the file:
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@@
 		(dnp no)
 		(fields_autoplaced yes)
-		(property "Reference" "SWD2"
+		(property "Reference" "SWD"
 			(at 170.18 86.3599 0)
 			(effects
@@
 			(project "PUTM_EV_DASHBOARD_SOCKET_2025"
 				(path "/8dcb9295-4fa2-433e-bd2f-4b006d008a4e/9b1bc52f-6033-4f71-8f99-a4060d1be2be"
-					(reference "SWD2")
+					(reference "SWD")
 					(unit 1)
 				)
