File: hardware/PUTM_EV_DASHBOARD_SOCKET_2025/CAN.kicad_sch (KiCad schematic)
At the start: 6 parts

Commit message: prawie gotowe
Parts:
- removed CAN0: Conn_01x04_MountingPin, Connector_Molex:Molex_CLIK-Mate_502382-0470_1x04-1MP_P1.25mm_Vertical, symbol Connector_Generic_MountingPin:Conn_01x04_MountingPin
- added CAN0: Conn_01x09, Connector_Dsub:DSUB-9_Pins_Horizontal_P2.77x2.84mm_EdgePinOffset4.94mm_Housed_MountingHolesOffset4.94mm, symbol Connector_Generic:Conn_01x09
- CAN1: footprint Connector_PinHeader_1.27mm:PinHeader_1x04_P1.27mm_Vertical -> Connector_Wire:SolderWire-0.1sqmm_1x04_P3.6mm_D0.4mm_OD1mm_Relief
Connections:
- net CAN1: now also CAN0.3 (Pin_3)
- net CAN2: now also CAN0.2 (Pin_2)
- net CAN3: now also CAN0.7 (Pin_7)
- net CAN4: now also CAN0.9 (Pin_9)
- new net GND: CAN0.8 (Pin_8)
- no-connect marks 0 -> 4
Changed lines of the file:
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@@
 	(generator_version "9.0")
 	(paper "A4")
+	(no_connect
+		(at 120.65 68.58)
+	)
+	(no_connect
+		(at 120.65 73.66)
+	)
+	(no_connect
+		(at 120.65 60.96)
+	)
+	(no_connect
+		(at 120.65 71.12)
+	)
 	(wire
 		(pts
@@
 	(wire
 		(pts
-			(xy 114.3 76.2) (xy 120.65 76.2)
+			(xy 114.3 63.5) (xy 120.65 63.5)
 		)
 		(stroke
@@
 	(global_label "CAN2"
 		(shape input)
-		(at 114.3 76.2 180)
+		(at 114.3 63.5 180)
 		(fields_autoplaced yes)
 		(effects
@@
 		)
 		(property "Intersheetrefs" "${INTERSHEET_REFS}"
-			(at 106.4162 76.2 0)
+			(at 106.4162 63.5 0)
 			(effects
 				(font
@@
 	(global_label "CAN3"
 		(shape input)
-		(at 120.65 78.74 180)
+		(at 120.65 76.2 180)
 		(fields_autoplaced yes)
 		(effects
@@
 		)
 		(property "Intersheetrefs" "${INTERSHEET_REFS}"
-			(at 112.7662 78.74 0)
+			(at 112.7662 76.2 0)
 			(effects
 				(font
@@
 	(global_label "CAN1"
 		(shape input)
-		(at 120.65 73.66 180)
+		(at 120.65 66.04 180)
 		(fields_autoplaced yes)
 		(effects
@@
 		)
 		(property "Intersheetrefs" "${INTERSHEET_REFS}"
-			(at 112.7662 73.66 0)
+			(at 112.7662 66.04 0)
 			(effects
 				(font
@@
 				(justify right)
 				(hide yes)
+			)
+		)
+	)
+	(symbol
+		(lib_id "Connector_Generic:Conn_01x09")
+		(at 125.73 71.12 0)
+		(unit 1)
+		(exclude_from_sim no)
+		(in_bom yes)
+		(on_board yes)
+		(dnp no)
+		(fields_autoplaced yes)
+		(property "Reference" "CAN0"
+			(at 128.27 69.8499 0)
+			(effects
+				(font
+					(size 1.27 1.27)
+				)
+				(justify left)
+			)
+		)
+		(property "Value" "Conn_01x09"
+			(at 128.27 72.3899 0)
+			(effects
+				(font
+					(size 1.27 1.27)
+				)
+				(justify left)
+			)
+		)
+		(property "Footprint" "Connector_Dsub:DSUB-9_Pins_Horizontal_P2.77x2.84mm_EdgePinOffset4.94mm_Housed_MountingHolesOffset4.94mm"
+			(at 125.73 71.12 0)
+			(effects
+				(font
+					(size 1.27 1.27)
+				)
+				(hide yes)
+			)
+		)
+		(property "Datasheet" "~"
+			(at 125.73 71.12 0)
+			(effects
+				(font
+					(size 1.27 1.27)
+				)
+				(hide yes)
+			)
+		)
+		(property "Description" "Generic connector, single row, 01x09, script generated (kicad-library-utils/schlib/autogen/connector/)"
+			(at 125.73 71.12 0)
+			(effects
+				(font
+					(size 1.27 1.27)
+				)
+				(hide yes)
+			)
+		)
+		(pin "8"
+		)
+		(pin "2"
+		)
+		(pin "5"
+		)
+		(pin "6"
+		)
+		(pin "9"
+		)
+		(pin "1"
+		)
+		(pin "3"
+		)
+		(pin "4"
+		)
+		(pin "7"
+		)
+		(instances
+			(project ""
+				(path "/8dcb9295-4fa2-433e-bd2f-4b006d008a4e/c92b4e8c-c56a-494c-81ca-99d15cc481d1"
+					(reference "CAN0")
+					(unit 1)
+				)
 			)
 		)
@@
 			)
 		)
-		(property "Footprint" "Connector_PinHeader_1.27mm:PinHeader_1x04_P1.27mm_Vertical"
+		(property "Footprint" "Connector_Wire:SolderWire-0.1sqmm_1x04_P3.6mm_D0.4mm_OD1mm_Relief"
 			(at 125.73 88.9 0)
 			(effects
@@
 	)
 	(symbol
-		(lib_name "Conn_01x04_MountingPin_1")
-		(lib_id "Connector_Generic_MountingPin:Conn_01x04_MountingPin")
-		(at 125.73 76.2 0)
+		(lib_id "power:GND")
+		(at 120.65 78.74 270)
 		(unit 1)
 		(exclude_from_sim no)
@@
 		(dnp no)
 		(fields_autoplaced yes)
-		(property "Reference" "CAN0"
-			(at 128.27 76.5555 0)
-			(effects
-				(font
-					(size 1.27 1.27)
-				)
-				(justify left)
-			)
-		)
-		(property "Value" "Conn_01x04_MountingPin"
-			(at 128.27 79.0955 0)
-			(effects
-				(font
-					(size 1.27 1.27)
-				)
-				(justify left)
-			)
-		)
-		(property "Footprint" "Connector_Molex:Molex_CLIK-Mate_502382-0470_1x04-1MP_P1.25mm_Vertical"
-			(at 125.73 76.2 0)
-			(effects
-				(font
-					(size 1.27 1.27)
-				)
-				(hide yes)
-			)
-		)
-		(property "Datasheet" "~"
-			(at 125.73 76.2 0)
-			(effects
-				(font
-					(size 1.27 1.27)
-				)
-				(hide yes)
-			)
-		)
-		(property "Description" "Generic connectable mounting pin connector, single row, 01x04, script generated (kicad-library-utils/schlib/autogen/connector/)"
-			(at 125.73 76.2 0)
+		(property "Reference" "#PWR039"
+			(at 114.3 78.74 0)
+			(effects
+				(font
+					(size 1.27 1.27)
+				)
+				(hide yes)
+			)
+		)
+		(property "Value" "GND"
+			(at 116.84 78.7399 90)
+			(effects
+				(font
+					(size 1.27 1.27)
+				)
+				(justify right)
+			)
+		)
+		(property "Footprint" ""
+			(at 120.65 78.74 0)
+			(effects
+				(font
+					(size 1.27 1.27)
+				)
+				(hide yes)
+			)
+		)
+		(property "Datasheet" ""
+			(at 120.65 78.74 0)
+			(effects
+				(font
+					(size 1.27 1.27)
+				)
+				(hide yes)
+			)
+		)
+		(property "Description" "Power symbol creates a global label with name \"GND\" , ground"
+			(at 120.65 78.74 0)
 			(effects
 				(font
@@
 		(pin "1"
 		)
-		(pin "4"
-		)
-		(pin "3"
-		)
-		(pin "2"
-		)
 		(instances
-			(project "PUTM_EV_DASHBOARD_SOCKET_2025"
+			(project ""
 				(path "/8dcb9295-4fa2-433e-bd2f-4b006d008a4e/c92b4e8c-c56a-494c-81ca-99d15cc481d1"
-					(reference "CAN0")
+					(reference "#PWR039")
 					(unit 1)
 				)

Commit message: jest jako tako
Parts:
- removed TERM_0: Conn_01x02_Pin, Connector_PinHeader_1.27mm:PinHeader_1x02_P1.27mm_Vertical, symbol Connector:Conn_01x02_Pin
- added D8: PESD2CAN.215, Package_TO_SOT_SMD:SOT-23-3, symbol BMS_LV_2022-rescue:D_TVS_x2_AAC-Device
- CAN0: footprint Connector_Dsub:DSUB-9_Pins_Horizontal_P2.77x2.84mm_EdgePinOffset4.94mm_Housed_MountingHolesOffset4.94mm -> Connector_Dsub:DSUB-9_Socket_Vertical_P2.77x2.84mm
Connections:
- net CAN2 is gone; now on net CAN_N: ALT_CAN0.1 (Pin_1), CAN0.2 (Pin_2), CAN1.2 (Pin_2)
- net GND: now also D8.3 (common)
- net CAN_N: now reaches R11.1
- net CAN_N: now also D8.2 (A2)
- net CAN1 renamed CAN_GND
- net CAN3 renamed CAN_P
- net CAN_P: now also D8.1 (A1)
- net CAN4 renamed CAN_VDD

Commit message: g3
Other:
- note added: "CAN NA ZŁĄCZU DB9"
- note added: "CAN PRZEWODOWY"
- moved on the sheet: ALT_CAN0, D8, R11, TERM_1
Changed lines of the file:
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@@
 	(generator_version "9.0")
 	(paper "A4")
+	(rectangle
+		(start 96.52 55.245)
+		(end 174.625 101.6)
+		(stroke
+			(width 0)
+			(type default)
+		)
+		(fill
+			(type none)
+		)
+	)
+	(rectangle
+		(start 175.895 60.96)
+		(end 230.505 98.425)
+		(stroke
+			(width 0)
+			(type default)
+		)
+		(fill
+			(type none)
+		)
+	)
+	(text "CAN PRZEWODOWY \n"
+		(exclude_from_sim no)
+		(at 192.278 64.516 0)
+		(effects
+			(font
+				(size 1.27 1.27)
+			)
+		)
+	)
+	(text "CAN NA ZŁĄCZU DB9\n"
+		(exclude_from_sim no)
+		(at 110.49 57.912 0)
+		(effects
+			(font
+				(size 1.27 1.27)
+			)
+		)
+	)
 	(no_connect
 		(at 120.65 68.58)
@@
 	(wire
 		(pts
-			(xy 231.14 90.17) (xy 231.14 87.63)
+			(xy 171.45 78.74) (xy 171.45 76.2)
 		)
 		(stroke
@@
 	(wire
 		(pts
-			(xy 194.31 87.63) (xy 194.31 92.71)
+			(xy 214.63 80.01) (xy 214.63 85.09)
 		)
 		(stroke
@@
 	(wire
 		(pts
-			(xy 194.31 80.01) (xy 194.31 82.55)
+			(xy 214.63 72.39) (xy 214.63 74.93)
 		)
 		(stroke
@@
 	(wire
 		(pts
-			(xy 231.14 87.63) (xy 228.6 87.63)
+			(xy 171.45 76.2) (xy 168.91 76.2)
 		)
 		(stroke
@@
 	(hierarchical_label "CAN_P"
 		(shape input)
-		(at 194.31 95.25 0)
+		(at 214.63 87.63 0)
 		(effects
 			(font
@@
 	(hierarchical_label "CAN_N"
 		(shape input)
-		(at 194.31 80.01 0)
+		(at 214.63 72.39 0)
 		(effects
 			(font
@@
 	(hierarchical_label "CAN_N"
 		(shape input)
-		(at 168.91 82.55 0)
+		(at 189.23 74.93 0)
 		(effects
 			(font
@@
 	(hierarchical_label "CAN_P"
 		(shape input)
-		(at 168.91 85.09 0)
+		(at 189.23 77.47 0)
 		(effects
 			(font
@@
 	(hierarchical_label "CAN_P"
 		(shape input)
-		(at 224.79 96.52 0)
+		(at 165.1 85.09 0)
 		(effects
 			(font
@@
 	(hierarchical_label "CAN_N"
 		(shape input)
-		(at 224.79 78.74 0)
+		(at 165.1 67.31 0)
 		(effects
 			(font
@@
 	(symbol
 		(lib_id "Connector:Conn_01x02_Pin")
-		(at 163.83 82.55 0)
+		(at 184.15 74.93 0)
 		(unit 1)
 		(exclude_from_sim no)
@@
 		(fields_autoplaced yes)
 		(property "Reference" "ALT_CAN0"
-			(at 164.465 77.47 0)
+			(at 184.785 69.85 0)
 			(effects
 				(font
@@
 		)
 		(property "Value" "Conn_01x02_Pin"
-			(at 164.465 80.01 0)
+			(at 184.785 72.39 0)
 			(effects
 				(font
@@
 		)
 		(property "Footprint" "Connector_Wire:SolderWire-0.1sqmm_1x02_P3.6mm_D0.4mm_OD1mm_Relief"
-			(at 163.83 82.55 0)
+			(at 184.15 74.93 0)
 			(effects
 				(font
@@
 		)
 		(property "Datasheet" "~"
-			(at 163.83 82.55 0)
+			(at 184.15 74.93 0)
 			(effects
 				(font
@@
 		)
 		(property "Description" "Generic connector, single row, 01x02, script generated"
-			(at 163.83 82.55 0)
+			(at 184.15 74.93 0)
 			(effects
 				(font
@@
 	(symbol
 		(lib_id "Device:R_Small")
-		(at 194.31 85.09 0)
+		(at 214.63 77.47 0)
 		(unit 1)
 		(exclude_from_sim no)
@@
 		(dnp no)
 		(property "Reference" "R11"
-			(at 196.85 83.8199 0)
+			(at 217.17 76.1999 0)
 			(effects
 				(font
@@
 		)
 		(property "Value" "120"
-			(at 196.596 85.598 0)
+			(at 216.916 77.978 0)
 			(effects
 				(font
@@
 		)
 		(property "Footprint" "Resistor_SMD:R_1206_3216Metric"
-			(at 194.31 85.09 0)
+			(at 214.63 77.47 0)
 			(effects
 				(font
@@
 		)
 		(property "Datasheet" "~"
-			(at 194.31 85.09 0)
+			(at 214.63 77.47 0)
 			(effects
 				(font
@@
 		)
 		(property "Description" "Resistor, small symbol"
-			(at 194.31 85.09 0)
+			(at 214.63 77.47 0)
 			(effects
 				(font
@@
 	(symbol
 		(lib_id "Connector:Conn_01x02_Pin")
-		(at 189.23 92.71 0)
+		(at 209.55 85.09 0)
 		(unit 1)
 		(exclude_from_sim no)
@@
 		(fields_autoplaced yes)
 		(property "Reference" "TERM_1"
-			(at 189.865 87.63 0)
+			(at 210.185 80.01 0)
 			(effects
 				(font
@@
 		)
 		(property "Value" "Conn_01x02_Pin"
-			(at 189.865 90.17 0)
+			(at 210.185 82.55 0)
 			(effects
 				(font
@@
 		)
 		(property "Footprint" "Connector_PinHeader_1.27mm:PinHeader_1x02_P1.27mm_Vertical"
-			(at 189.23 92.71 0)
+			(at 209.55 85.09 0)
 			(effects
 				(font
@@
 		)
 		(property "Datasheet" "~"
-			(at 189.23 92.71 0)
+			(at 209.55 85.09 0)
 			(effects
 				(font
@@
 		)
 		(property "Description" "Generic connector, single row, 01x02, script generated"
-			(at 189.23 92.71 0)
+			(at 209.55 85.09 0)
 			(effects
 				(font
@@
 	(symbol
 		(lib_id "BMS_LV_2022-rescue:D_TVS_x2_AAC-Device")
-		(at 224.79 87.63 90)
+		(at 165.1 76.2 90)
 		(unit 1)
 		(exclude_from_sim no)
@@
 		(dnp no)
 		(property "Reference" "D8"
-			(at 218.44 88.9 0)
+			(at 158.75 77.47 0)
 			(effects
 				(font
@@
 		)
 		(property "Value" "PESD2CAN.215"
-			(at 220.98 95.25 0)
+			(at 161.29 83.82 0)
 			(effects
 				(font
@@
 		)
 		(property "Footprint" "Package_TO_SOT_SMD:SOT-23-3"
-			(at 224.79 91.44 0)
+			(at 165.1 80.01 0)
 			(effects
 				(font
@@
 		)
 		(property "Datasheet" "https://assets.nexperia.com/documents/data-sheet/PESD2CAN.pdf"
-			(at 224.79 91.44 0)
+			(at 165.1 80.01 0)
 			(effects
 				(font
@@
 		)
 		(property "Description" ""
-			(at 224.79 87.63 0)
+			(at 165.1 76.2 0)
 			(effects
 				(font
@@
 		)
 		(property "Mouser Price/Stock" "https://www.mouser.pl/ProductDetail/Nexperia/PESD2CAN215?qs=LOCUfHb8d9sqg7TaLUP2JQ%3D%3D"
-			(at 224.79 87.63 0)
+			(at 165.1 76.2 0)
 			(effects
 				(font
@@
 		)
 		(property "Author" ""
-			(at 224.79 87.63 0)
+			(at 165.1 76.2 0)
 			(effects
 				(font
@@
 		)
 		(property "License" ""
-			(at 224.79 87.63 0)
+			(at 165.1 76.2 0)
 			(effects
 				(font
@@
 		)
 		(property "MPN" ""
-			(at 224.79 87.63 0)
+			(at 165.1 76.2 0)
 			(effects
 				(font
@@
 		)
 		(property "Manufacturer" ""
-			(at 224.79 87.63 0)
+			(at 165.1 76.2 0)
 			(effects
 				(font
@@
 		)
 		(property "Sim.Pins" ""
-			(at 224.79 87.63 0)
+			(at 165.1 76.2 0)
 			(effects
 				(font
@@
 		(lib_name "GND_1")
 		(lib_id "power:GND")
-		(at 231.14 90.17 0)
+		(at 171.45 78.74 0)
 		(unit 1)
 		(exclude_from_sim no)
@@
 		(fields_autoplaced yes)
 		(property "Reference" "#PWR043"
-			(at 231.14 96.52 0)
+			(at 171.45 85.09 0)
 			(effects
 				(font
@@
 		)
 		(property "Value" "GND"
-			(at 231.14 95.25 0)
+			(at 171.45 83.82 0)
 			(effects
 				(font
@@
 		)
 		(property "Footprint" ""
-			(at 231.14 90.17 0)
+			(at 171.45 78.74 0)
 			(effects
 				(font
@@
 		)
 		(property "Datasheet" ""
-			(at 231.14 90.17 0)
+			(at 171.45 78.74 0)
 			(effects
 				(font
@@
 		)
 		(property "Description" "Power symbol creates a global label with name \"GND\" , ground"
-			(at 231.14 90.17 0)
-			(effects
-				(font
+			(at 171.45 78.74 0)
+			(effects
+				(font

Commit message: fixed button logic, holes for inserts, distance from mounting holes to P4 socket, changed jumpers, TVS diode and footprint for laboratory socket 4m
Parts:
- removed D8: PESD2CAN.215, Package_TO_SOT_SMD:SOT-23-3, symbol BMS_LV_2022-rescue:D_TVS_x2_AAC-Device
- added D24: PESD2IVN24-U, Package_TO_SOT_SMD:SOT-323_SC-70, symbol Device:D_TVS_Dual_AAC
- TERM_1: footprint Connector_PinHeader_1.27mm:PinHeader_1x02_P1.27mm_Vertical -> Connector_PinHeader_2.54mm:PinHeader_1x02_P2.54mm_Vertical
Connections:
- net CAN_N: now also D24.2 (A2)
- net CAN_P: now also D24.1 (A1)
- net GND: now also D24.3 (common)
Changed lines of the file:
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@@
+	)
+	(symbol
+		(lib_id "Device:D_TVS_Dual_AAC")
+		(at 165.1 76.2 90)
+		(unit 1)
+		(exclude_from_sim no)
+		(in_bom yes)
+		(on_board yes)
+		(dnp no)
+		(property "Reference" "D24"
+			(at 160.02 77.47 0)
+			(effects
+				(font
+					(size 1.27 1.27)
+				)
+				(justify left)
+			)
+		)
+		(property "Value" "PESD2IVN24-U"
+			(at 162.56 76.2 0)
+			(effects
+				(font
+					(size 1.27 1.27)
+				)
+			)
+		)
+		(property "Footprint" "Package_TO_SOT_SMD:SOT-323_SC-70"
+			(at 165.1 80.01 0)
+			(effects
+				(font
+					(size 1.27 1.27)
+				)
+				(hide yes)
+			)
+		)
+		(property "Datasheet" "~"
+			(at 165.1 80.01 0)
+			(effects
+				(font
+					(size 1.27 1.27)
+				)
+				(hide yes)
+			)
+		)
+		(property "Description" ""
+			(at 165.1 76.2 0)
+			(effects
+				(font
+					(size 1.27 1.27)
+				)
+				(hide yes)
+			)
+		)
+		(pin "1"
+		)
+		(pin "2"
+		)
+		(pin "3"
+		)
+		(instances
+			(project "PUTM_EV_DASHBOARD_SOCKET_2025"
+				(path "/8dcb9295-4fa2-433e-bd2f-4b006d008a4e/c92b4e8c-c56a-494c-81ca-99d15cc481d1"
+					(reference "D24")
+					(unit 1)
+				)
+			)
+		)
 	)
 	(symbol
@@
 			)
 		)
-		(property "Footprint" "Connector_PinHeader_1.27mm:PinHeader_1x02_P1.27mm_Vertical"
+		(property "Footprint" "Connector_PinHeader_2.54mm:PinHeader_1x02_P2.54mm_Vertical"
 			(at 209.55 85.09 0)
 			(effects
@@
 					(unit 1)
 				)
-			)
-		)
-	)
-	(symbol
-		(lib_id "BMS_LV_2022-rescue:D_TVS_x2_AAC-Device")
-		(at 165.1 76.2 90)
-		(unit 1)
-		(exclude_from_sim no)
-		(in_bom yes)
-		(on_board yes)
-		(dnp no)
-		(property "Reference" "D8"
-			(at 158.75 77.47 0)
-			(effects
-				(font
-					(size 1.27 1.27)
-				)
-				(justify left)
-			)
-		)
-		(property "Value" "PESD2CAN.215"
-			(at 161.29 83.82 0)
-			(effects
-				(font
-					(size 1.27 1.27)
-				)
-				(justify left)
-			)
-		)
-		(property "Footprint" "Package_TO_SOT_SMD:SOT-23-3"
-			(at 165.1 80.01 0)
-			(effects
-				(font
-					(size 1.27 1.27)
-				)
-				(hide yes)
-			)
-		)
-		(property "Datasheet" "https://assets.nexperia.com/documents/data-sheet/PESD2CAN.pdf"
-			(at 165.1 80.01 0)
-			(effects
-				(font
-					(size 1.27 1.27)
-				)
-				(hide yes)
-			)
-		)
-		(property "Description" ""
-			(at 165.1 76.2 0)
-			(effects
-				(font
-					(size 1.27 1.27)
-				)
-				(hide yes)
-			)
-		)
-		(property "Mouser Price/Stock" "https://www.mouser.pl/ProductDetail/Nexperia/PESD2CAN215?qs=LOCUfHb8d9sqg7TaLUP2JQ%3D%3D"
-			(at 165.1 76.2 0)
-			(effects
-				(font
-					(size 1.27 1.27)
-				)
-				(hide yes)
-			)
-		)
-		(property "Author" ""
-			(at 165.1 76.2 0)
-			(effects
-				(font
-					(size 1.27 1.27)
-				)
-			)
-		)
-		(property "License" ""
-			(at 165.1 76.2 0)
-			(effects
-				(font
-					(size 1.27 1.27)
-				)
-			)
-		)
-		(property "MPN" ""
-			(at 165.1 76.2 0)
-			(effects
-				(font
-					(size 1.27 1.27)
-				)
-			)
-		)
-		(property "Manufacturer" ""
-			(at 165.1 76.2 0)
-			(effects
-				(font
-					(size 1.27 1.27)
-				)
-			)
-		)
-		(property "Sim.Pins" ""
-			(at 165.1 76.2 0)
-			(effects
-				(font
-					(size 1.27 1.27)
-				)
-			)
-		)
-		(pin "3"
-		)
-		(pin "2"
-		)
-		(pin "1"
-		)
-		(instances
-			(project "PUTM_EV_DASHBOARD_SOCKET_2025"
-				(path "/8dcb9295-4fa2-433e-bd2f-4b006d008a4e/c92b4e8c-c56a-494c-81ca-99d15cc481d1"
-					(reference "D8")
-					(unit 1)
-				)
